File: Vectorblade_PLCC32_THT.kicad_sch (KiCad schematic)
At the start: 5 parts, among them CON3 EDGE-CONNECTOR, U1 SST39SF020, U2 74AHC1G08, U3 74AHC1G04

Commit message: I forgot to connect A15
Shame !
Connections:
- net V-A15: now also CON3.16 (CE)
- no-connect marks 6 -> 5
Changed lines of the file:
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@@
   (junction (at 100.33 35.56) (diameter 0) (color 0 0 0 0)
   )
-  (no_connect (at 127 66.04))
   (no_connect (at 127 71.12))
   (no_connect (at 127 73.66))
@@
     (stroke (width 0) (type default) (color 0 0 0 0))
   )
+  (bus_entry (at 137.16 66.04) (size 2.54 2.54)
+    (stroke (width 0) (type default) (color 0 0 0 0))
+  )
   (wire (pts (xy 245.11 60.96) (xy 245.11 63.5))
     (stroke (width 0) (type default) (color 0 0 0 0))
@@
   )
   (wire (pts (xy 68.58 71.12) (xy 76.2 71.12))
+    (stroke (width 0) (type default) (color 0 0 0 0))
+  )
+  (wire (pts (xy 127 66.04) (xy 137.16 66.04))
     (stroke (width 0) (type default) (color 0 0 0 0))
   )
@@
     (effects (font (size 1.2446 1.2446)) (justify left bottom))
   )
+  (label "V-A15" (at 137.16 66.04 180)
+    (effects (font (size 1.27 1.27)) (justify right bottom))
+  )
   (symbol (lib_id "74xGxx:74AHC1G08") (at 157.48 124.46 0) (unit 1)
