File: Vectorblade_PLCC32_THT_Kicad7.kicad_pcb (KiCad board)
At the start: 2 copper layers, 47.2 x 46.9 mm, 12 parts, among them CON3 EDGE-CONNECTOR, U1 SST39SF020, U2 74AHC1G08, U3 74AHC1G04

Commit message: Update Gerber
Other:
- board text added: "v1.2"
- board text removed: "v1.1"
